File: plate-top/AK62-plate-top.kicad_pcb (KiCad board)
At the start: 2 copper layers, 276.2 x 95.2 mm, 0 parts

Commit message: update plate
Other:
- board text added: "AK62 / Apple Keyboard M0116 Mod PCB Designed by Ryo Nakae"
Changed lines of the file:
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@@
   (general
     (thickness 1.6)
-    (drawings 1215)
+    (drawings 1216)
     (tracks 0)
     (zones 0)
@@
     (uvia_dia 0.3)
     (uvia_drill 0.1)
+  )
+  (gr_text "AK62 / Apple Keyboard M0116 Mod\nPCB Designed by Ryo Nakae" (at 139.27 -2.16) (layer F.Mask)
+    (effects (font (size 1.5 1.5) (thickness 0.3)))
   )
   (gr_circle (center 179.32 -90.49) (end 179.32 -89.39) (layer Edge.Cuts) (width 0.05))
@@
     (polygon
       (pts
-        (xy -3.24 -104.73) (xy -3.24 5.93) (xy 293.63 5.93) (xy 293.63 -102.96)
+        (xy 0 -99.06) (xy 0 10.16) (xy 292.1 10.16) (xy 292.1 -99.06)
       )
     )
@@
     (polygon
       (pts
-        (xy -1.19065 -104.7772) (xy -1.19065 6.90577) (xy 293.61429 6.90577) (xy 293.61429 -104.06281)
+        (xy 0 -99.06) (xy 0 10.16) (xy 292.1 10.16) (xy 292.1 -99.06)
       )
     )
